Commit message: update model with static RG3 gripper

File: urdf/ur3_joint_limited_robot.urdf.xacro (robot description, xacro)
@@ -7,4 +7,6 @@
   <!-- ur3 -->
   <xacro:include filename="$(find ur_description)/urdf/ur3.urdf.xacro" />
+  <!-- gripper RG2 -->
+  <xacro:include filename="$(find ur_description)/urdf/rg2.urdf.xacro" />
   <!-- arm -->
   <xacro:arg name="kinematics_config" default="$(find ur_description)/config/ur3_default.yaml"/>
@@ -24,4 +26,5 @@
     <child link = "base_link" />
     <origin xyz="0.0 0.0 0.0" rpy="0.0 0.0 0.0" />
-  </joint>
+</joint>
+<xacro:rg2 parent="ee_link" />
 </robot>

File: urdf/ur3_robot.urdf.xacro (robot description, xacro)
@@ -7,4 +7,6 @@
   <!-- ur3 -->
   <xacro:include filename="$(find ur_description)/urdf/ur3.urdf.xacro" />
+  <!-- gripper -->
+  <xacro:include filename="$(find ur_description)/urdf/rg2.urdf.xacro" />
   <!-- arm -->
   <xacro:arg name="kinematics_config" default="$(find ur_description)/config/ur3_default.yaml"/>
@@ -18,4 +20,5 @@
     <child link = "base_link" />
     <origin xyz="0.0 0.0 0.0" rpy="0.0 0.0 0.0" />
-  </joint>
+</joint>
+    <xacro:rg2 parent="ee_link" />
 </robot>
