Commit message: latest update with gazebo grasp fix plugin

File: urdf/rg2.gazebo.xacro (robot description, xacro)
@@ -4,5 +4,5 @@
 	<!-- Hand -->
 	<gazebo reference="hand_link">
-		<mu1>0.2</mu1>
+        <mu1>0.2</mu1>
 		<mu2>0.2</mu2>
 		<material>Gazebo/DarkGrey</material>
@@ -22,7 +22,10 @@
 		<selfCollide>false</selfCollide>
 	</gazebo>
-	<gazebo reference="l_finger_link">
-		<mu1>0.2</mu1>
-		<mu2>0.2</mu2>
+    <gazebo reference="l_finger_link">
+        <minDepth>0.003</minDepth>
+        <maxVel>0.0</maxVel>
+        <mu1>100</mu1>
+        <mu2>100</mu2>
+        <kp>100000</kp>
 		<material>Gazebo/FlatBlack</material>
 		<selfCollide>false</selfCollide>
@@ -41,7 +44,10 @@
 		<selfCollide>false</selfCollide>
 	</gazebo>
-	<gazebo reference="r_finger_link">
-		<mu1>0.2</mu1>
-		<mu2>0.2</mu2>
+    <gazebo reference="r_finger_link">
+        <minDepth>0.003</minDepth>
+        <maxVel>0.00</maxVel>
+        <mu1>100</mu1>
+        <mu2>100</mu2>
+        <kp>100000</kp>
 		<material>Gazebo/FlatBlack</material>
 		<selfCollide>false</selfCollide>

File: urdf/rg2.transmissions.xacro (robot description, xacro)
@@ -8,5 +8,5 @@
 			</joint>
 			<actuator name="${name}_motor">
-				<hardwareInterface>hardware_interface/PositionJointInterface</hardwareInterface>
+                <!-- <hardwareInterface>hardware_interface/PositionJointInterface</hardwareInterface> -->
 				<mechanicalReduction>1</mechanicalReduction>
 			</actuator>

File: urdf/rg2.urdf.xacro (robot description, xacro)
@@ -270,4 +270,23 @@
             </inertial>
         </link>
+        <!--
+        <gazebo>
+            <plugin name="gazebo_grasp_fix" filename="libgazebo_grasp_fix.so">
+                <arm>
+                    <arm_name>robot</arm_name>
+                    <palm_link>hand_link</palm_link>
+                    <gripper_link>l_finger_link</gripper_link>
+                    <gripper_link>r_finger_link</gripper_link>
+                </arm>
+                <force_angle_tolerance>100</force_angle_tolerance>
+                <update_rate>4</update_rate>
+                <grip_count_threshold>4</grip_count_threshold>
+                <max_grip_count>8</max_grip_count>
+                <release_tolerance>0.005</release_tolerance>
+                <disable_collision_on_attach>false</disable_collision_on_attach>
+                <contact_topic>__default_topic__</contact_topic>
+            </plugin>
+        </gazebo>
+        -->
     </xacro:macro>
 </robot>

File: urdf/ur3.urdf.xacro (robot description, xacro)
@@ -50,6 +50,6 @@
         <xacro:property name="upper_arm_inertia_offset" value="0.12" />  <!-- measured from model -->
         <!-- This is for compatibility reasons, as transformation between base and base_link was always 180 degree in the ur_description -->
-        <xacro:property name="base_correction" value="${pi}" />
-        <link name="${prefix}base_link" >
+    <xacro:property name="base_correction" value="${pi}" />
+    <link name="${prefix}base_link" >
             <visual>
                 <origin xyz="0 0 0" rpy="0 0 ${base_correction}"/>
@@ -306,15 +306,15 @@
         </link>
         <joint name="${prefix}ee_fixed_joint" type="fixed">
-            <parent link="${prefix}wrist_3_link" />
+            <parent link="${prefix}tool0" />
             <child link = "${prefix}ee_link" />
-            <origin xyz="0.0 0.0 0.0" rpy="0.0 ${-pi/2.0} ${pi/2.0}" />
+            <origin xyz="0.0 0.0 0.17" rpy="0.0 0.0 0.0" />
         </joint>
         <link name="${prefix}ee_link">
-            <collision>
+            <!-- <collision>
                     <geometry>
                         <box size="0.01 0.01 0.01"/>
                     </geometry>
-                    <origin rpy="0 0 0" xyz="-0.01 0 0"/>
-            </collision>
+                    <origin rpy="0 0 0" xyz="0 0 0"/>
+            </collision> -->
         </link>
         <joint name="${prefix}wrist_3_passive_joint" type="fixed">
@@ -326,14 +326,16 @@
         <xacro:ur_arm_gazebo prefix="${prefix}" />
         <!-- ROS base_link to UR 'Base' Coordinates transform -->
-        <link name="${prefix}base"/>
-        <joint name="${prefix}base_link-base_fixed_joint" type="fixed">
+        <!-- <link name="${prefix}base"/> -->
+        <!--
+        <joint name="${prefix}base_link-base_fixed_joint" type="fixed"> -->
             <!-- NOTE: this rotation is only needed as long as base_link itself is
                         not corrected wrt the real robot (ie: rotated over 180
                         degrees)
             -->
+            <!--
             <origin xyz="0 0 0" rpy="0 0 ${-base_correction}"/>
             <parent link="${prefix}base_link"/>
             <child link="${prefix}base"/>
-        </joint>
+        </joint> -->
         <!-- Frame coincident with all-zeros TCP on UR controller -->
         <link name="${prefix}tool0"/>

File: urdf/ur3_joint_limited_robot.urdf.xacro (robot description, xacro)
@@ -34,4 +34,5 @@
     <!-- UR to Gripper -->
     <xacro:rg2 parent="tool0" />
+    <!--
     <joint name="end_effector_fixed_joint" type="fixed">
         <parent link="tool0" />
@@ -41,3 +42,21 @@
     <link name="end_effector_link">
     </link>
+    -->
+    <gazebo>
+        <plugin name="gazebo_grasp_fix" filename="libgazebo_grasp_fix.so">
+            <arm>
+                <arm_name>ur3</arm_name>
+                <palm_link>wrist_3_link</palm_link>
+                <gripper_link>l_finger_link</gripper_link>
+                <gripper_link>r_finger_link</gripper_link>
+            </arm>
+            <forces_angle_tolerance>90</forces_angle_tolerance>
+            <update_rate>4</update_rate>
+            <grip_count_threshold>2</grip_count_threshold>
+            <max_grip_count>4</max_grip_count>
+            <release_tolerance>0.005</release_tolerance>
+            <disable_collisions_on_attach>false</disable_collisions_on_attach>
+            <contact_topic>__default_topic__</contact_topic>
+        </plugin>
+    </gazebo>
 </robot>

File: urdf/ur3_robot.urdf.xacro (robot description, xacro)
@@ -27,3 +27,13 @@
     <!-- UR to Gripper -->
     <xacro:rg2 parent="tool0" />
+    <gazebo>
+        <plugin name="gazebo+grasp_fix" filename="libgazebo_grasp_fix.so">
+            <arm>
+                <arm_name>ur3_arm</arm_name>
+                <palm_link>hand_link</palm_link>
+                <gripper_link>l_finger_link</gripper_link>
+                <gripper_link>r_finger_link</gripper_link>
+            </arm>
+        </plugin>
+    </gazebo>
 </robot>
